File: pcb/pcb.kicad_sch (KiCad schematic)
At the start: 0 parts

Commit message: not finished
Parts:
- added C? (x2): 22pF, symbol Device:C_Small
- added C? (x3): 0.1uF, symbol Device:C_Small
- added C?: 1uF, symbol Device:C_Small
- added C?: 10uF, symbol Device:C_Small
- added R? (x2): 22, symbol Device:R_Small
- added R? (x2): 10k, symbol Device:R_Small
- added SW?: SW_Push, symbol Switch:SW_Push
- added U?: ATmega32U4-A, Package_QFP:TQFP-44_10x10mm_P0.8mm, symbol MCU_Microchip_ATmega:ATmega32U4-A
- added Y?: Crystal_GND24_Small, symbol Device:Crystal_GND24_Small
Connections:
- new net: C?.2, U?.17 (XTAL1), Y?.1
- new net: C?.2, U?.16 (XTAL2), Y?.3
- new net: R?.2, U?.4 (D+)
- new net: C?.1, U?.6 (UCAP)
- new net: R?.2, SW?.2, U?.13 (~{RESET})
- new net: R?.2, U?.3 (D-)
- new net: R?.2, U?.33 (~{HWB}/PE2)
- new net +5V: C?.1, C?.1, C?.1, C?.1, R?.1, U?.14 (VCC), U?.2 (UVCC), U?.24 (AVCC), U?.34 (VCC), U?.44 (AVCC), U?.7 (VBUS)
- new net D+: R?.1
- new net D-: R?.1
- new net GND: C?.1, C?.1, C?.2, C?.2, C?.2, C?.2, C?.2, R?.1, SW?.1, U?.15 (GND), U?.23 (GND), U?.35 (GND), U?.43 (GND), U?.5 (UGND), Y?.2, Y?.4
